File: Power.kicad_sch (KiCad schematic)
At the start: 0 parts

Commit message: created esp32 s3 mini connection to rp2350 added SD card Routed them together
Parts:
- added C20: 100n, Capacitor_SMD:C_0805_2012Metric_Pad1.18x1.45mm_HandSolder, symbol Device:C
- added C21, C22: 47u, Capacitor_SMD:C_0805_2012Metric_Pad1.18x1.45mm_HandSolder, symbol Device:C
- added D3, D4: D, Diode_SMD:D_0805_2012Metric, symbol Device:D
- added F1: JK-SMD0805-020-30V, EasyEDA:F0805, symbol EasyEDA:JK-SMD0805-020-30V
- added L2: FTC252010S4R7MBCA, EasyEDA:IND-SMD_L2.5-W2.0-VLS252012CX-150M, symbol EasyEDA:FTC252010S4R7MBCA
- added Power: LED, LED_SMD:LED_0805_2012Metric, symbol Device:LED
- added R12: 1k, Resistor_SMD:R_0805_2012Metric, symbol Device:R
- added U7: AP63205WU, Package_TO_SOT_SMD:TSOT-23-6_HandSoldering, symbol Regulator_Switching:AP63205WU
Connections:
- new net: Power.1 (K), R12.1
- new net: C21.1, D3.1 (K), U7.2 (EN), U7.3 (IN)
- new net: C22.1, D4.2 (A), L2.2, U7.1 (FB)
- new net: C20.1, L2.1, U7.5 (SW)
- new net: C20.2, U7.6 (BST)
- new net: D4.1 (K), F1.1
- new net +5V: F1.2, Power.2 (A)
- new net GND: C21.2, C22.2, R12.2, U7.4 (GND)
- new net VSS: D3.2 (A)
Other:
- note added: "? should i add a turn off switch?"

Commit message: generated pdf
Parts:
- added C4, C5: 47u, Capacitor_SMD:C_0805_2012Metric_Pad1.18x1.45mm_HandSolder, symbol Device:C
- added C6: 100n, Capacitor_SMD:C_0805_2012Metric_Pad1.18x1.45mm_HandSolder, symbol Device:C
- added U4: AMS1117-3.3, Package_TO_SOT_SMD:SOT-223-3_TabPin2, symbol Regulator_Linear:AMS1117-3.3
Connections:
- net +5V: now also C4.1, U4.3 (VI)
- net GND: now also C4.2, C5.2, C6.2, U4.1 (GND)
- new net +3V3: C5.1, C6.1, U4.2 (VO)
Other:
- moved on the sheet: C20, C21, C22, D3, D4, F1, L2, Power, R12, U7
